File: source_files/PCB/hackpad.kicad_pcb (KiCad board)
At the start: 2 copper layers, 80 x 62 mm, 18 parts, among them J1 Conn_01x04, SW1 SW_Push, SW2 SW_Push, SW3 SW_Push, SW4 SW_Push, SW5 SW_Push, SW6 SW_Push, SW7 SW_Push, SW8 RotaryEncoder_Switch, U1 MOUDLE-SEEEDUINO-XIAO

Commit message: Add files via upload
Connections:
- U1 pad 10: ROTB -> COL1
- U1 pad 11: ROTA -> COL0
- U1 pad 3: unconnected-(U1-PA10_A2_D2-Pad3) -> ROTA
- U1 pad 4: COL0 -> ROTB
- U1 pad 5: COL1 -> SDA
- U1 pad 6: COL2 -> SCL
- U1 pad 7: COL3 -> unconnected-(U1-PB08_A6_D6_TX-Pad7)
- U1 pad 8: SDA -> COL3
- U1 pad 9: SCL -> COL2
Routing:
- net ROTB: track 96.6 -> 16.8 mm
- net COL0: track 112.5 -> 94.3 mm
- net ROW1: track 98.4 -> 82.8 mm
- net ROW0: track 106.7 -> 91.7 mm
- net COL1: track 68.1 -> 81.8 mm
- net COL2: track 57.0 -> 70.3 mm
- net ROTA: track 27.1 -> 14.8 mm
- net GND: track 50.4 -> 42.6 mm
- net SDA: track 16.2 -> 11.0 mm
- net Net-(D1-A): track 14.6 -> 12.5 mm
- net SCL: track 11.9 -> 13.5 mm
- net COL3: track 47.3 -> 48.0 mm
